File: C64UserBreakout.kicad_pcb (KiCad board)
At the start: 2 copper layers, 58 x 85.5 mm, 490 parts, among them CON1 C64-UserPort-Sym, J1 Power, J2 GND, J3 Breakout1, J4 Breakout2, SW1 Reset

Commit message: Mostly finied layout for rev 1.
Parts:
- added G***: LOGO, Logo:bigby2-cu, F.Cu at (155.1, 61.2)
- J1: value Power -> Power1; footprint Connector_PinHeader_2.54mm:PinHeader_2x02_P2.54mm_Vertical -> C64UserBreakout:PinHeader_2x02_Power
- J2: value GND -> Power2; footprint Connector_PinHeader_2.54mm:PinHeader_1x02_P2.54mm_Vertical -> C64UserBreakout:PinHeader_2x02_Power
- moved H1 19.8 mm to (137.2, 68.6)
- moved J2 13.0 mm to (144.8, 71.1), turned to 0 degrees
- moved SW1 8.38 mm to (158.2, 68.6)
Connections:
- J2 pad 1: GND -> +5V
- J2 pad 2: GND -> +5V
Routing:
- net RST: track 83.9 -> 86.6 mm
- net GND: track 214.7 -> 217.0 mm
- net /FLAG2: track 95.2 -> 97.4 mm
- net /PA2: track 85.9 -> 83.8 mm
- net /PB2: track 94.6 -> 93.1 mm
- net /PB1: track 96.0 -> 94.5 mm
- net /PB0: track 97.4 -> 96.0 mm
- net /PB6: track 88.7 -> 87.3 mm
- net /ATN: track 93.4 -> 92.0 mm
- net /9VAC1: track 94.8 -> 93.6 mm
- net /9VAC2: track 96.2 -> 95.0 mm
- net /PB4: track 90.5 -> 89.3 mm
- net /CNT1: track 84.9 -> 86.1 mm
- net /PB5: track 90.6 -> 89.9 mm
Other:
- net class AC added: clearance 0.25, trace_width 0.35, via_dia 0.8, via_drill 0.4
- board text added: "+5V"
- board text added: "9VAC1"
- board text added: "9VAC2"
- board text added: "ATN"
- board text added: "CNT1"
- board text added: "CNT2"
- board text added: "FLAG2"
- board text added: "GND"
- board text added: "PA2"
- board text added: "PB0"
- board text added: "PB1"
- board text added: "PB2"
- board text added: "PB3"
- board text added: "PB4"
- board text added: "PB5"
- board text added: "PB6"
- board text added: "PB7"
- board text added: "PC2"
- board text added: "RST"
- board text added: "SP1"
- board text added: "SP2"
- board text added: "THIS SIDE UP"
- board text added: "github.com/hackup/C64UserBreakout Rev.1"
